Commit message: robot core xacro fix

File: description/robot_core.xacro (robot description, xacro)
@@ -27,5 +27,5 @@
             <origin xyz="0 0 0" />
             <geometry>
-                <mesh filename="file://$(find kapibara)/meshes/Bottom.stl" scale="0.001 0.001 0.001" />
+                <mesh filename="file://$(find kapibara_robot)/meshes/Bottom.stl" scale="0.001 0.001 0.001" />
             </geometry>
             <material name="black" />
@@ -42,5 +42,5 @@
             <origin xyz="0 0 0.05" />
             <geometry>
-                <mesh filename="file://$(find kapibara)/meshes/Top.stl" scale="0.001 0.001 0.001" />
+                <mesh filename="file://$(find kapibara_robot)/meshes/Top.stl" scale="0.001 0.001 0.001" />
             </geometry>
             <material name="orange" />
